File: pcb/shortkeyboard.kicad_sch (KiCad schematic)
At the start: 96 parts, among them SW1 SW_Push, SW10 SW_Push, SW11 SW_Push, SW12 SW_Push, SW13 SW_Push, SW14 SW_Push, SW15 SW_Push, SW16 SW_Push, SW17 SW_Push, SW18 SW_Push, SW19 SW_Push, SW2 SW_Push, SW20 SW_Push, SW21 SW_Push, SW22 SW_Push, SW23 SW_Push, SW24 SW_Push, SW25 SW_Push, SW26 SW_Push, SW27 SW_Push, SW28 SW_Push, SW29 SW_Push, SW3 SW_Push, SW30 SW_Push, SW31 SW_Push, SW32 SW_Push, SW33 SW_Push, SW34 SW_Push, SW35 SW_Push, SW36 SW_Push, SW37 SW_Push, SW38 SW_Push, SW39 SW_Push, SW4 SW_Push, SW40 SW_Push, SW41 SW_Push, SW42 SW_Push, SW43 SW_Push, SW44 SW_Push, SW45 SW_Push, SW46 SW_Push, SW47 SW_Push, SW5 SW_Push, SW6 SW_Push, SW7 SW_Push, SW8 SW_Push, SW9 SW_Push, U1 nice_nano

Commit message: placement in pcb
Parts:
- SW31: footprint Button_Switch_Keyboard:SW_Cherry_MX_2.00u_PCB -> Button_Switch_Keyboard:SW_Cherry_MX_1.00u_PCB
- SW42: footprint Button_Switch_Keyboard:SW_Cherry_MX_1.00u_PCB -> Button_Switch_Keyboard:SW_Cherry_MX_2.00u_PCB
Connections:
- net BATT+: now also U1.13 (BAT+)
- no-connect marks 0 -> 6
Changed lines of the file:
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@@
 	)
 	(junction
-		(at 26.67 40.64)
-		(diameter 0)
-		(color 0 0 0 0)
-	)
-	(junction
 		(at 255.27 57.15)
 		(diameter 0)
@@
 	)
 	(junction
-		(at 26.67 38.1)
-		(diameter 0)
-		(color 0 0 0 0)
-	)
-	(junction
 		(at 138.43 45.72)
 		(diameter 0)
@@
 		(color 0 0 0 0)
 	)
+	(no_connect
+		(at 85.09 45.72)
+	)
+	(no_connect
+		(at 85.09 43.18)
+	)
+	(no_connect
+		(at 66.04 66.04)
+	)
+	(no_connect
+		(at 63.5 66.04)
+	)
+	(no_connect
+		(at 60.96 66.04)
+	)
+	(no_connect
+		(at 85.09 38.1)
+	)
 	(wire
 		(pts
@@
 	(wire
 		(pts
+			(xy 46.99 38.1) (xy 27.94 38.1)
+		)
+		(stroke
+			(width 0)
+			(type default)
+		)
+	)
+	(wire
+		(pts
 			(xy 151.13 45.72) (xy 163.83 45.72)
 		)
@@
 	(wire
 		(pts
-			(xy 26.67 38.1) (xy 26.67 40.64)
-		)
-		(stroke
-			(width 0)
-			(type default)
-		)
-	)
-	(wire
-		(pts
 			(xy 151.13 83.82) (xy 163.83 83.82)
 		)
@@
 	(wire
 		(pts
-			(xy 26.67 40.64) (xy 46.99 40.64)
+			(xy 255.27 38.1) (xy 255.27 57.15)
 		)
 		(stroke
@@
 	(wire
 		(pts
-			(xy 255.27 38.1) (xy 255.27 57.15)
+			(xy 179.07 38.1) (xy 179.07 57.15)
 		)
 		(stroke
@@
 	(wire
 		(pts
-			(xy 179.07 38.1) (xy 179.07 57.15)
+			(xy 176.53 102.87) (xy 189.23 102.87)
 		)
 		(stroke
@@
 	(wire
 		(pts
-			(xy 176.53 102.87) (xy 189.23 102.87)
+			(xy 204.47 76.2) (xy 204.47 95.25)
 		)
 		(stroke
@@
 	(wire
 		(pts
-			(xy 204.47 76.2) (xy 204.47 95.25)
+			(xy 163.83 64.77) (xy 176.53 64.77)
 		)
 		(stroke
@@
 	(wire
 		(pts
-			(xy 163.83 64.77) (xy 176.53 64.77)
+			(xy 115.57 57.15) (xy 115.57 76.2)
 		)
 		(stroke
@@
 	(wire
 		(pts
-			(xy 115.57 57.15) (xy 115.57 76.2)
+			(xy 35.56 43.18) (xy 35.56 40.64)
 		)
 		(stroke
@@
 	(wire
 		(pts
-			(xy 26.67 30.48) (xy 26.67 38.1)
-		)
-		(stroke
-			(width 0)
-			(type default)
-		)
-	)
-	(wire
-		(pts
 			(xy 191.77 25.4) (xy 191.77 38.1)
 		)
@@
 	(wire
 		(pts
-			(xy 46.99 38.1) (xy 26.67 38.1)
+			(xy 27.94 38.1) (xy 27.94 43.18)
 		)
 		(stroke
@@
 	(wire
 		(pts
-			(xy 46.99 30.48) (xy 26.67 30.48)
+			(xy 46.99 30.48) (xy 17.78 30.48)
 		)
 		(stroke
@@
 	(wire
 		(pts
-			(xy 26.67 44.45) (xy 26.67 40.64)
+			(xy 17.78 30.48) (xy 17.78 35.56)
 		)
 		(stroke
@@
 		)
 	)
+	(wire
+		(pts
+			(xy 35.56 40.64) (xy 46.99 40.64)
+		)
+		(stroke
+			(width 0)
+			(type default)
+		)
+	)
 	(global_label "COL11"
 		(shape input)
@@
 		)
 	)
+	(global_label "BATT+"
+		(shape input)
+		(at 85.09 33.02 0)
+		(fields_autoplaced yes)
+		(effects
+			(font
+				(size 1.27 1.27)
+			)
+			(justify left)
+		)
+		(property "Intersheetrefs" "${INTERSHEET_REFS}"
+			(at 93.9414 33.02 0)
+			(hide yes)
+			(show_name no)
+			(do_not_autoplace no)
+			(effects
+				(font
+					(size 1.27 1.27)
+				)
+				(justify left)
+			)
+		)
+	)
 	(global_label "COL6"
 		(shape input)
@@
 			)
 		)
-		(property "Footprint" "Button_Switch_Keyboard:SW_Cherry_MX_1.00u_PCB"
+		(property "Footprint" "Button_Switch_Keyboard:SW_Cherry_MX_2.00u_PCB"
 			(at 184.15 90.17 0)
 			(hide yes)
@@
 			)
 		)
-		(property "Footprint" "Button_Switch_Keyboard:SW_Cherry_MX_2.00u_PCB"
+		(property "Footprint" "Button_Switch_Keyboard:SW_Cherry_MX_1.00u_PCB"
 			(at 196.85 71.12 0)
 			(hide yes)
@@
 	)
 	(symbol
+		(lib_id "power:GND")
+		(at 35.56 43.18 0)
+		(unit 1)
+		(body_style 1)
+		(exclude_from_sim no)
+		(in_bom yes)
+		(on_board yes)
+		(in_pos_files yes)
+		(dnp no)
+		(fields_autoplaced yes)
+		(property "Reference" "#PWR05"
+			(at 35.56 49.53 0)
+			(hide yes)
+			(show_name no)
+			(do_not_autoplace no)
+			(effects
+				(font
+					(size 1.27 1.27)
+				)
+			)
+		)
+		(property "Value" "GND"
+			(at 35.56 48.26 0)
+			(show_name no)
+			(do_not_autoplace no)
+			(effects
+				(font
+					(size 1.27 1.27)
+				)
+			)
+		)
+		(property "Footprint" ""
+			(at 35.56 43.18 0)
+			(hide yes)
+			(show_name no)
+			(do_not_autoplace no)
+			(effects
+				(font
+					(size 1.27 1.27)
+				)
+			)
+		)
+		(property "Datasheet" ""
+			(at 35.56 43.18 0)
+			(hide yes)
+			(show_name no)
+			(do_not_autoplace no)
+			(effects
+				(font
+					(size 1.27 1.27)
+				)
+			)
+		)
+		(property "Description" "Power symbol creates a global label with name \"GND\" , ground"
+			(at 35.56 43.18 0)
+			(hide yes)
+			(show_name no)
+			(do_not_autoplace no)
+			(effects
+				(font
+					(size 1.27 1.27)
+				)
+			)
+		)
+		(pin "1"
+		)
+		(instances
+			(project "shortkeyboard"
+				(path "/2210a0b6-eb5a-42d3-9315-02ed508503ff"
+					(reference "#PWR05")
+					(unit 1)
+				)
+			)
+		)
+	)
+	(symbol
 		(lib_id "Switch:SW_Push")
 		(at 222.25 57.15 0)
@@
 	(symbol
 		(lib_id "power:GND")
-		(at 26.67 44.45 0)
+		(at 17.78 35.56 0)
 		(unit 1)
 		(body_style 1)
@@
 		(fields_autoplaced yes)
 		(property "Reference" "#PWR01"
-			(at 26.67 50.8 0)
+			(at 17.78 41.91 0)
 			(hide yes)
 			(show_name no)
@@
 		)
 		(property "Value" "GND"
-			(at 26.67 49.53 0)
+			(at 17.78 40.64 0)
 			(show_name no)
 			(do_not_autoplace no)
@@
 		)
 		(property "Footprint" ""
-			(at 26.67 44.45 0)
+			(at 17.78 35.56 0)
 			(hide yes)
 			(show_name no)
@@
 		)
 		(property "Datasheet" ""
-			(at 26.67 44.45 0)
+			(at 17.78 35.56 0)
 			(hide yes)
 			(show_name no)
@@
 		)
 		(property "Description" "Power symbol creates a global label with name \"GND\" , ground"
-			(at 26.67 44.45 0)
+			(at 17.78 35.56 0)
 			(hide yes)
 			(show_name no)
@@
 					(unit 1)
 				)
+			)
+		)
+	)
+	(symbol
+		(lib_id "power:GND")
+		(at 27.94 43.18 0)
+		(unit 1)
+		(body_style 1)
+		(exclude_from_sim no)
+		(in_bom yes)
+		(on_board yes)
+		(in_pos_files yes)
+		(dnp no)
+		(fields_autoplaced yes)
+		(property "Reference" "#PWR06"
+			(at 27.94 49.53 0)
+			(hide yes)
+			(show_name no)
+			(do_not_autoplace no)
+			(effects
+				(font
+					(size 1.27 1.27)
+				)
+			)
+		)
+		(property "Value" "GND"
+			(at 27.94 48.26 0)
+			(show_name no)
+			(do_not_autoplace no)
+			(effects
+				(font
+					(size 1.27 1.27)
+				)
+			)
+		)
+		(property "Footprint" ""
+			(at 27.94 43.18 0)
+			(hide yes)
+			(show_name no)
+			(do_not_autoplace no)
+			(effects
+				(font
+					(size 1.27 1.27)
+				)
+			)
+		)
+		(property "Datasheet" ""
+			(at 27.94 43.18 0)
+			(hide yes)
+			(show_name no)
+			(do_not_autoplace no)
+			(effects
+				(font
+					(size 1.27 1.27)
+				)
+			)
+		)
+		(property "Description" "Power symbol creates a global label with name \"GND\" , ground"
+			(at 27.94 43.18 0)
+			(hide yes)
+			(show_name no)
+			(do_not_autoplace no)
+			(effects
+				(font
+					(size 1.27 1.27)
+				)
+			)
+		)
+		(pin "1"
+		)
+		(instances
+			(project "shortkeyboard"
+				(path "/2210a0b6-eb5a-42d3-9315-02ed508503ff"
+					(reference "#PWR06")
+					(unit 1)
+				)

Commit message: added 0.91 oled
Parts:
- added U2: ER_OLEDM0.91_1x-I2C, Display:ER_OLEDM0.91_1x-I2C, symbol Display_Graphic:ER_OLEDM0.91_1x-I2C
Connections:
- net +3V3: now also U2.2 (VCC)
- net GND: now also U2.1 (GND)
- net OLED_SCL: now reaches U1.17 (P0.31-LF)
- net OLED_SCL: now also U2.3 (SCL)
- net OLED_SDA: now reaches U1.18 (P0.29-LF)
- net OLED_SDA: now also U2.4 (SDA)
- no-connect marks 6 -> 4

Commit message: schematic of led
Parts:
- added C1: 100nF, Capacitor_THT:C_Disc_D5.0mm_W2.5mm_P5.00mm, symbol Device:C
- added C2: 100uF, Capacitor_THT:CP_Radial_D5.0mm_P2.00mm, symbol Device:C
- added D48, D49, D50, D51, D52, D53, D54, D55, D56, D57, D58, D59, D60, D61, D62, D63, D64, D65, D66, D67, D68, D69, D70, D71, D72, D73, D74, D75, D76, D77, D78, D79, D80, D81, D82, D83, D84, D85, D86, D87, D88, D89, D90, D91, D92, D93, D94: SK6812MINI-E, LED_SMD:LED_SK6812MINI-E_3.2x2.8mm_P1.5mm_ReverseMount, symbol LED:SK6812MINI-E
- added R1: 330Ω, Resistor_SMD:R_0805_2012Metric_Pad1.20x1.40mm_HandSolder, symbol Device:R
- added U3: SN74AHCT125N, SN74AHCT125N:DIP794W45P254L1930H508Q14, symbol SN74AHCT125N:SN74AHCT125N
Connections:
- net GND: now also C1.2, C2.1, D48.1 (VSS), D49.1 (VSS), D50.1 (VSS), D51.1 (VSS), D52.1 (VSS), D53.1 (VSS), D54.1 (VSS), D55.1 (VSS), D56.1 (VSS), D57.1 (VSS), D58.1 (VSS), D59.1 (VSS), D60.1 (VSS), D61.1 (VSS), D62.1 (VSS), D63.1 (VSS), D64.1 (VSS), D65.1 (VSS), D66.1 (VSS), D67.1 (VSS), D68.1 (VSS), D69.1 (VSS), D70.1 (VSS), D71.1 (VSS), D72.1 (VSS), D73.1 (VSS), D74.1 (VSS), D75.1 (VSS), D76.1 (VSS), D77.1 (VSS), D78.1 (VSS), D79.1 (VSS), D80.1 (VSS), D81.1 (VSS), D82.1 (VSS), D83.1 (VSS), D84.1 (VSS), D85.1 (VSS), D86.1 (VSS), D87.1 (VSS), D88.1 (VSS), D89.1 (VSS), D90.1 (VSS), D91.1 (VSS), D92.1 (VSS), D93.1 (VSS), D94.1 (VSS), U3.1 (1~{OE}), U3.7 (GND)
- net LED_DOUT: now reaches U1.25 (P1.01-LF)
- net LED_DOUT: now also U3.2 (1A)
- new net: D89.4 (DOUT), D90.2 (DIN)
- new net: D90.4 (DOUT), D91.2 (DIN)
- new net: D79.4 (DOUT), D80.2 (DIN)
- new net: D80.4 (DOUT), D81.2 (DIN)
- new net: D48.4 (DOUT), D49.2 (DIN)
- new net: D49.4 (DOUT), D50.2 (DIN)
- new net: D59.4 (DOUT), D60.2 (DIN)
- new net: D60.4 (DOUT), D61.2 (DIN)
- new net: D54.4 (DOUT), D55.2 (DIN)
- new net: D55.4 (DOUT), D56.2 (DIN)
- new net: D74.4 (DOUT), D75.2 (DIN)
- new net: D75.4 (DOUT), D76.2 (DIN)
- new net: D56.4 (DOUT), D57.2 (DIN)
- new net: D57.4 (DOUT), D58.2 (DIN)
- new net: D85.4 (DOUT), D86.2 (DIN)
- new net: D86.4 (DOUT), D87.2 (DIN)
- new net: D63.4 (DOUT), D64.2 (DIN)
- new net: D64.4 (DOUT), D65.2 (DIN)
- new net: D76.4 (DOUT), D77.2 (DIN)
- new net: D77.4 (DOUT), D78.2 (DIN)
- new net: D73.4 (DOUT), D74.2 (DIN)
- new net: D93.4 (DOUT), D94.2 (DIN)
- new net: D78.4 (DOUT), D79.2 (DIN)
- new net: D67.4 (DOUT), D68.2 (DIN)
- new net: D68.4 (DOUT), D69.2 (DIN)
- new net: D58.4 (DOUT), D59.2 (DIN)
- new net: D81.4 (DOUT), D82.2 (DIN)
- new net: D71.4 (DOUT), D72.2 (DIN)
- new net: D72.4 (DOUT), D73.2 (DIN)
- new net: D87.4 (DOUT), D88.2 (DIN)
- new net: D84.4 (DOUT), D85.2 (DIN)
- new net: R1.2, U3.3 (1Y)
- new net: D70.4 (DOUT), D71.2 (DIN)
- new net: D65.4 (DOUT), D66.2 (DIN)
- new net: D62.4 (DOUT), D63.2 (DIN)
- new net: D52.4 (DOUT), D53.2 (DIN)
- new net: D53.4 (DOUT), D54.2 (DIN)
- new net: D66.4 (DOUT), D67.2 (DIN)
- new net: D82.4 (DOUT), D83.2 (DIN)
- new net: D83.4 (DOUT), D84.2 (DIN)
- new net: D91.4 (DOUT), D92.2 (DIN)
- new net: D92.4 (DOUT), D93.2 (DIN)
- new net: D51.4 (DOUT), D52.2 (DIN)
- new net: D69.4 (DOUT), D70.2 (DIN)
- new net: D50.4 (DOUT), D51.2 (DIN)
- new net: D88.4 (DOUT), D89.2 (DIN)
- new net: D61.4 (DOUT), D62.2 (DIN)
- new net +5V: C1.1, C2.2
- new net LED_DIN: D48.2 (DIN), R1.1
- new net VCC: D48.3 (VDD), D49.3 (VDD), D50.3 (VDD), D51.3 (VDD), D52.3 (VDD), D53.3 (VDD), D54.3 (VDD), D55.3 (VDD), D56.3 (VDD), D57.3 (VDD), D58.3 (VDD), D59.3 (VDD), D60.3 (VDD), D61.3 (VDD), D62.3 (VDD), D63.3 (VDD), D64.3 (VDD), D65.3 (VDD), D66.3 (VDD), D67.3 (VDD), D68.3 (VDD), D69.3 (VDD), D70.3 (VDD), D71.3 (VDD), D72.3 (VDD), D73.3 (VDD), D74.3 (VDD), D75.3 (VDD), D76.3 (VDD), D77.3 (VDD), D78.3 (VDD), D79.3 (VDD), D80.3 (VDD), D81.3 (VDD), D82.3 (VDD), D83.3 (VDD), D84.3 (VDD), D85.3 (VDD), D86.3 (VDD), D87.3 (VDD), D88.3 (VDD), D89.3 (VDD), D90.3 (VDD), D91.3 (VDD), D92.3 (VDD), D93.3 (VDD), D94.3 (VDD), U3.14 (VCC)
- no-connect marks 4 -> 6
Other:
- moved on the sheet: BT1
