File: pcb/shortkeyboard.kicad_pcb (KiCad board)
At the start: 2 copper layers, 96 parts, among them SW1 SW_Push, SW10 SW_Push, SW11 SW_Push, SW12 SW_Push, SW13 SW_Push, SW14 SW_Push, SW15 SW_Push, SW16 SW_Push, SW17 SW_Push, SW18 SW_Push, SW19 SW_Push, SW2 SW_Push, SW20 SW_Push, SW21 SW_Push, SW22 SW_Push, SW23 SW_Push, SW24 SW_Push, SW25 SW_Push, SW26 SW_Push, SW27 SW_Push, SW28 SW_Push, SW29 SW_Push, SW3 SW_Push, SW30 SW_Push, SW31 SW_Push, SW32 SW_Push, SW33 SW_Push, SW34 SW_Push, SW35 SW_Push, SW36 SW_Push, SW37 SW_Push, SW38 SW_Push, SW39 SW_Push, SW4 SW_Push, SW40 SW_Push, SW41 SW_Push, SW42 SW_Push, SW43 SW_Push, SW44 SW_Push, SW45 SW_Push, SW46 SW_Push, SW47 SW_Push, SW5 SW_Push, SW6 SW_Push, SW7 SW_Push, SW8 SW_Push, SW9 SW_Push, U1 nice_nano

Commit message: routing done
Parts:
- moved U1 267.3 mm to (110.9, 75.8), turned to 90 degrees
- moved BT1 262.6 mm to (135.7, 70.5)
Routing:
- net ROW3: track 0.00 -> 313.4 mm
- net ROW2: track 0.00 -> 277.8 mm
- net COL11: track 0.00 -> 268.4 mm
- net ROW1: track 0.00 -> 263.3 mm
- net ROW0: track 0.00 -> 245.3 mm
- net COL10: track 0.00 -> 245.1 mm
- net COL9: track 0.00 -> 213.2 mm
- net COL8: track 0.00 -> 196.7 mm
- net COL7: track 0.00 -> 180.1 mm
- net COL5: track 0.00 -> 151.0 mm
- net COL6: track 0.00 -> 144.5 mm
- net COL4: track 0.00 -> 132.0 mm
- net COL3: track 0.00 -> 115.6 mm
- net COL2: track 0.00 -> 99.5 mm
- net COL1: track 0.00 -> 88.1 mm
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Other:
- board outline added: 234.1 x 102 mm

Commit message: added 0.91 oled
Parts:
- added U2: ER_OLEDM0.91_1x-I2C, Display:ER_OLEDM0.91_1x-I2C, F.Cu at (280.6, 78.3)
Connections:
- U1 pad 17: unconnected-(U1-P0.31-LF-Pad17) -> OLED_SCL
- U1 pad 18: unconnected-(U1-P0.29-LF-Pad18) -> OLED_SDA
Routing:
- net +3V3: track 0.00 -> 180.6 mm
- net OLED_SCL: track 0.00 -> 175.6 mm, vias 0 -> 1
- net OLED_SDA: track 0.00 -> 173.9 mm, vias 0 -> 3
- net GND: track 65.2 -> 211.2 mm
Other:
- outline, holes or cut-outs redrawn

Commit message: schematic of led
Parts:
- added C1: 100nF, Capacitor_THT:C_Disc_D5.0mm_W2.5mm_P5.00mm, F.Cu at (385.2, 102.5)
- added C2: 100uF, Capacitor_THT:CP_Radial_D5.0mm_P2.00mm, F.Cu at (386.0, 107.8)
- added D48: SK6812MINI-E, LED_SMD:LED_SK6812MINI-E_3.2x2.8mm_P1.5mm_ReverseMount, F.Cu at (345.7, 82.0)
- added D49: SK6812MINI-E, LED_SMD:LED_SK6812MINI-E_3.2x2.8mm_P1.5mm_ReverseMount, F.Cu at (345.7, 86.9)
- added D50: SK6812MINI-E, LED_SMD:LED_SK6812MINI-E_3.2x2.8mm_P1.5mm_ReverseMount, F.Cu at (345.7, 91.8)
- added D51: SK6812MINI-E, LED_SMD:LED_SK6812MINI-E_3.2x2.8mm_P1.5mm_ReverseMount, F.Cu at (345.7, 96.6)
- added D52: SK6812MINI-E, LED_SMD:LED_SK6812MINI-E_3.2x2.8mm_P1.5mm_ReverseMount, F.Cu at (345.7, 101.5)
- added D53: SK6812MINI-E, LED_SMD:LED_SK6812MINI-E_3.2x2.8mm_P1.5mm_ReverseMount, F.Cu at (345.7, 106.4)
- added D54: SK6812MINI-E, LED_SMD:LED_SK6812MINI-E_3.2x2.8mm_P1.5mm_ReverseMount, F.Cu at (345.7, 111.2)
- added D55: SK6812MINI-E, LED_SMD:LED_SK6812MINI-E_3.2x2.8mm_P1.5mm_ReverseMount, F.Cu at (345.7, 116.1)
- added D56: SK6812MINI-E, LED_SMD:LED_SK6812MINI-E_3.2x2.8mm_P1.5mm_ReverseMount, F.Cu at (345.7, 121.0)
- added D57: SK6812MINI-E, LED_SMD:LED_SK6812MINI-E_3.2x2.8mm_P1.5mm_ReverseMount, F.Cu at (345.7, 125.9)
- added D58: SK6812MINI-E, LED_SMD:LED_SK6812MINI-E_3.2x2.8mm_P1.5mm_ReverseMount, F.Cu at (354.1, 82.0)
- added D59: SK6812MINI-E, LED_SMD:LED_SK6812MINI-E_3.2x2.8mm_P1.5mm_ReverseMount, F.Cu at (354.1, 86.9)
- added D60: SK6812MINI-E, LED_SMD:LED_SK6812MINI-E_3.2x2.8mm_P1.5mm_ReverseMount, F.Cu at (354.1, 91.8)
- added D61: SK6812MINI-E, LED_SMD:LED_SK6812MINI-E_3.2x2.8mm_P1.5mm_ReverseMount, F.Cu at (354.1, 96.6)
- added D62: SK6812MINI-E, LED_SMD:LED_SK6812MINI-E_3.2x2.8mm_P1.5mm_ReverseMount, F.Cu at (354.1, 101.5)
- added D63: SK6812MINI-E, LED_SMD:LED_SK6812MINI-E_3.2x2.8mm_P1.5mm_ReverseMount, F.Cu at (354.1, 106.4)
- added D64: SK6812MINI-E, LED_SMD:LED_SK6812MINI-E_3.2x2.8mm_P1.5mm_ReverseMount, F.Cu at (354.1, 111.2)
- added D65: SK6812MINI-E, LED_SMD:LED_SK6812MINI-E_3.2x2.8mm_P1.5mm_ReverseMount, F.Cu at (354.1, 116.1)
- added D66: SK6812MINI-E, LED_SMD:LED_SK6812MINI-E_3.2x2.8mm_P1.5mm_ReverseMount, F.Cu at (354.1, 121.0)
- added D67: SK6812MINI-E, LED_SMD:LED_SK6812MINI-E_3.2x2.8mm_P1.5mm_ReverseMount, F.Cu at (354.1, 125.9)
- added D68: SK6812MINI-E, LED_SMD:LED_SK6812MINI-E_3.2x2.8mm_P1.5mm_ReverseMount, F.Cu at (362.6, 82.0)
- added D69: SK6812MINI-E, LED_SMD:LED_SK6812MINI-E_3.2x2.8mm_P1.5mm_ReverseMount, F.Cu at (362.6, 86.9)
- added D70: SK6812MINI-E, LED_SMD:LED_SK6812MINI-E_3.2x2.8mm_P1.5mm_ReverseMount, F.Cu at (362.6, 91.8)
- added D71: SK6812MINI-E, LED_SMD:LED_SK6812MINI-E_3.2x2.8mm_P1.5mm_ReverseMount, F.Cu at (362.6, 96.6)
- added D72: SK6812MINI-E, LED_SMD:LED_SK6812MINI-E_3.2x2.8mm_P1.5mm_ReverseMount, F.Cu at (362.6, 101.5)
- added D73: SK6812MINI-E, LED_SMD:LED_SK6812MINI-E_3.2x2.8mm_P1.5mm_ReverseMount, F.Cu at (362.6, 106.4)
- added D74: SK6812MINI-E, LED_SMD:LED_SK6812MINI-E_3.2x2.8mm_P1.5mm_ReverseMount, F.Cu at (362.6, 111.2)
- added D75: SK6812MINI-E, LED_SMD:LED_SK6812MINI-E_3.2x2.8mm_P1.5mm_ReverseMount, F.Cu at (362.6, 116.1)
- added D76: SK6812MINI-E, LED_SMD:LED_SK6812MINI-E_3.2x2.8mm_P1.5mm_ReverseMount, F.Cu at (362.6, 121.0)
- added D77: SK6812MINI-E, LED_SMD:LED_SK6812MINI-E_3.2x2.8mm_P1.5mm_ReverseMount, F.Cu at (362.6, 125.9)
- added D78: SK6812MINI-E, LED_SMD:LED_SK6812MINI-E_3.2x2.8mm_P1.5mm_ReverseMount, F.Cu at (371.0, 82.0)
- added D79: SK6812MINI-E, LED_SMD:LED_SK6812MINI-E_3.2x2.8mm_P1.5mm_ReverseMount, F.Cu at (371.0, 86.9)
- added D80: SK6812MINI-E, LED_SMD:LED_SK6812MINI-E_3.2x2.8mm_P1.5mm_ReverseMount, F.Cu at (371.0, 91.8)
- added D81: SK6812MINI-E, LED_SMD:LED_SK6812MINI-E_3.2x2.8mm_P1.5mm_ReverseMount, F.Cu at (371.0, 96.6)
- added D82: SK6812MINI-E, LED_SMD:LED_SK6812MINI-E_3.2x2.8mm_P1.5mm_ReverseMount, F.Cu at (371.0, 101.5)
- added D83: SK6812MINI-E, LED_SMD:LED_SK6812MINI-E_3.2x2.8mm_P1.5mm_ReverseMount, F.Cu at (371.0, 106.4)
- added D84: SK6812MINI-E, LED_SMD:LED_SK6812MINI-E_3.2x2.8mm_P1.5mm_ReverseMount, F.Cu at (371.0, 111.2)
- added D85: SK6812MINI-E, LED_SMD:LED_SK6812MINI-E_3.2x2.8mm_P1.5mm_ReverseMount, F.Cu at (371.0, 116.1)
- added D86: SK6812MINI-E, LED_SMD:LED_SK6812MINI-E_3.2x2.8mm_P1.5mm_ReverseMount, F.Cu at (371.0, 121.0)
- added D87: SK6812MINI-E, LED_SMD:LED_SK6812MINI-E_3.2x2.8mm_P1.5mm_ReverseMount, F.Cu at (371.0, 125.9)
- added D88: SK6812MINI-E, LED_SMD:LED_SK6812MINI-E_3.2x2.8mm_P1.5mm_ReverseMount, F.Cu at (379.4, 82.0)
- added D89: SK6812MINI-E, LED_SMD:LED_SK6812MINI-E_3.2x2.8mm_P1.5mm_ReverseMount, F.Cu at (379.4, 86.9)
- added D90: SK6812MINI-E, LED_SMD:LED_SK6812MINI-E_3.2x2.8mm_P1.5mm_ReverseMount, F.Cu at (379.4, 91.8)
- added D91: SK6812MINI-E, LED_SMD:LED_SK6812MINI-E_3.2x2.8mm_P1.5mm_ReverseMount, F.Cu at (379.4, 96.6)
- added D92: SK6812MINI-E, LED_SMD:LED_SK6812MINI-E_3.2x2.8mm_P1.5mm_ReverseMount, F.Cu at (379.4, 101.5)
- added D93: SK6812MINI-E, LED_SMD:LED_SK6812MINI-E_3.2x2.8mm_P1.5mm_ReverseMount, F.Cu at (379.4, 106.4)
- added D94: SK6812MINI-E, LED_SMD:LED_SK6812MINI-E_3.2x2.8mm_P1.5mm_ReverseMount, F.Cu at (379.4, 111.2)
- added R1: 330Ω, Resistor_SMD:R_0805_2012Metric_Pad1.20x1.40mm_HandSolder, F.Cu at (386.0, 112.5)
- added U3: SN74AHCT125N, SN74AHCT125N:DIP794W45P254L1930H508Q14, F.Cu at (389.6, 90.0)
Connections:
- U1 pad 25: unconnected-(U1-P1.01-LF-Pad25) -> LED_DOUT

Commit message: added led to the switches, routing done
Parts:
- D48, D49, D50, D51, D52, D53, D54, D55, D56, D57, D58, D59, D60, D61, D62, D63, D64, D65, D66, D67, D68, D69, D70, D71, D72, D73, D74, D75, D76, D77, D78, D79, D80, D81, D82, D83, D84, D85, D86, D87, D88, D89, D90, D91, D92, D93, D94: moved to B.Cu
- moved D84 272.8 mm to (102.7, 160.6)
- moved D72 263.0 mm to (102.7, 141.5)
- moved D60 253.3 mm to (102.7, 122.5)
- moved D85 253.2 mm to (121.7, 160.6)
- moved D48 244.0 mm to (102.7, 103.4)
- moved D73 243.4 mm to (121.7, 141.6)
- moved D61 233.8 mm to (121.8, 122.5)
- moved D86 233.6 mm to (140.8, 160.6)
- moved R1 232.5 mm to (156.1, 77.5)
- moved D49 224.6 mm to (121.7, 103.4)
- moved D74 223.8 mm to (140.8, 141.5)
- moved U3 220.0 mm to (170.3, 72.8), turned to 90 degrees
- moved D88 215.3 mm to (178.9, 160.6)
- moved D62 214.4 mm to (140.8, 122.5)
- moved D87 214.0 mm to (159.9, 160.6)
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Routing:
- net VCC: track 0.00 -> 1077.4 mm, vias 0 -> 13
- net Net-(D59-DOUT): track 0.00 -> 246.3 mm
- net Net-(D71-DOUT): track 0.00 -> 245.5 mm
- net Net-(D83-DOUT): track 0.00 -> 245.4 mm, vias 0 -> 2
- net LED_DIN: track 0.00 -> 85.9 mm, vias 0 -> 5
- net LED_DOUT: track 0.00 -> 49.8 mm, vias 0 -> 2
- net Net-(D89-DOUT): track 0.00 -> 23.8 mm
- net Net-(D88-DOUT): track 0.00 -> 23.7 mm
- net Net-(D60-DOUT): track 0.00 -> 14.3 mm
- net Net-(D66-DOUT): track 0.00 -> 14.3 mm
- net Net-(D49-DOUT): track 0.00 -> 14.3 mm
- net Net-(D54-DOUT): track 0.00 -> 14.3 mm
- net Net-(D52-DOUT): track 0.00 -> 14.2 mm
- net Net-(D79-DOUT): track 0.00 -> 14.2 mm
- net Net-(D64-DOUT): track 0.00 -> 14.2 mm
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- added copper zone on B.Cu, net GND
